Commit message: Add joy

File: install/daramg_sim/share/daramg_sim/urdf/2Dlidar.xacro (robot description, xacro)
@@ -1,64 +1 @@
-<?xml version="1.0"?>
-<robot xmlns:xacro="http://www.ros.org/wiki/xacro" name="robot_name">
-    <!-- STEP 10 - Lidar -->
-    <joint type="fixed" name="scan_joint">
-        <origin xyz="0.25 0 0.25" rpy="0 0 0"/>
-        <child link="scan_link"/>
-        <parent link="base_link"/>
-        <axis xyz="0 1 0" rpy="0 0 0"/>
-    </joint>
-    <link name='scan_link'>
-        <xacro:inertial_box mass="1e-5" x=".1" y=".1" z=".1">
-            <origin xyz="0 0 0" rpy="0 0 0"/>
-        </xacro:inertial_box>
-        <collision name='collision'>
-            <origin xyz="0 0 0" rpy="0 0 0"/>
-            <geometry>
-                <box size=".1 .1 .1"/>
-            </geometry>
-        </collision>
-        <visual name='scan_link_visual'>
-            <origin xyz="0 0 0" rpy="0 0 0"/>
-            <geometry>
-                <box size=".1 .1 .1"/>
-            </geometry>
-        </visual>
-    </link>
-  <gazebo reference="scan_link">
-    <sensor name="gpu_lidar" type="gpu_lidar">
-      <update_rate>10</update_rate>
-      <topic>scan</topic>
-      <gz_frame_id>scan_link</gz_frame_id>
-      <lidar>
-        <scan>
-          <horizontal>
-            <samples>720</samples>
-            <!--(max_angle-min_angle)/samples * resolution -->
-            <resolution>1</resolution>
-            <min_angle>-3.14156</min_angle>
-            <max_angle>3.14156</max_angle>
-          </horizontal>
-          <!-- Dirty hack for fake lidar detections with ogre 1 rendering in VM -->
-          <!-- <vertical>
-              <samples>3</samples>
-              <min_angle>-0.001</min_angle>
-              <max_angle>0.001</max_angle>
-          </vertical> -->
-        </scan>
-        <range>
-          <min>0.05</min>
-          <max>10.0</max>
-          <resolution>0.01</resolution>
-        </range>
-        <noise>
-            <type>gaussian</type>
-            <mean>0.0</mean>
-            <stddev>0.01</stddev>
-        </noise>
-        <frame_id>scan_link</frame_id>
-      </lidar>
-      <always_on>1</always_on>
-      <visualize>true</visualize>
-    </sensor>
-  </gazebo>
-</robot>
+/home/kimhoyun/DARAM-G/src/daramg_sim/urdf/2Dlidar.xacro

File: install/daramg_sim/share/daramg_sim/urdf/RGB_D.xacro (robot description, xacro)
@@ -1,80 +1 @@
-<?xml version="1.0"?>
-<robot xmlns:xacro="http://www.ros.org/wiki/xacro" name="robot_name">
-    <!-- STEP 10 - Lidar -->
-    <joint name="depth_pillar_joint" type="fixed">
-        <origin xyz="0.15 0.0 0.275" rpy="0.0 0.0 0.0"/>
-        <parent link="base_link"/>
-        <child link="depth_pillar"/>
-        <axis xyz="0.0 0.0 0.0"/>
-        <limit lower="0.0" upper="0.0" effort="0.0" velocity="0.0"/>
-    </joint>
-    <link name="depth_pillar">
-        <xacro:inertial_box mass="0.5" x=".1" y=".1" z=".15">
-            <origin xyz="0 0 0" rpy="0 0 0"/>
-        </xacro:inertial_box>
-        <visual>
-            <origin xyz="0.0 0.0 0.0" rpy="0.0 0.0 0.0"/>
-            <geometry>
-                <box size="0.1 0.1 0.15"/>
-            </geometry>
-            <material name="green"/>
-        </visual>
-        <collision>
-            <origin xyz="0.0 0.0 0.0" rpy="0.0 0.0 0.0"/>
-            <geometry>
-                <box size="0.1 0.1 0.15"/>
-            </geometry>
-        </collision>
-    </link>
-    <joint type="fixed" name="depth_joint">
-        <origin xyz="0.0 0 0.125" rpy="0 0 0"/>
-        <child link="depth_link"/>
-        <parent link="depth_pillar"/>
-        <axis xyz="0 1 0" rpy="0 0 0"/>
-    </joint>
-    <link name='depth_link'>
-        <xacro:inertial_box mass="1e-5" x=".1" y=".15" z=".1">
-            <origin xyz="0 0 0" rpy="0 0 0"/>
-        </xacro:inertial_box>
-        <collision name='collision'>
-            <origin xyz="0 0 0" rpy="0 0 0"/>
-            <geometry>
-                <box size=".1 .15 .1"/>
-            </geometry>
-        </collision>
-        <visual name='depth_link_visual'>
-            <origin xyz="0 0 0" rpy="0 0 0"/>
-            <geometry>
-                <box size=".1 .15 .1"/>
-            </geometry>
-        </visual>
-    </link>
-    <joint type="fixed" name="camera_optical_joint">
-        <origin xyz="0 0 0" rpy="-1.5707 0 -1.5707"/>
-        <child link="camera_link_optical"/>
-        <parent link="depth_link"/>
-    </joint>
-    <link name="camera_link_optical">
-    </link>
-  <gazebo reference="depth_link">
-    <sensor name="rgbd_camera" type="rgbd_camera">
-      <camera>
-        <horizontal_fov>1.25</horizontal_fov>
-        <image>
-          <width>320</width>
-          <height>240</height>
-        </image>
-        <clip>
-          <near>0.3</near>
-          <far>15</far>
-        </clip>
-        <optical_frame_id>depth_link</optical_frame_id>
-      </camera>
-      <always_on>1</always_on>
-      <update_rate>20</update_rate>
-      <visualize>true</visualize>
-      <topic>camera</topic>
-      <gz_frame_id>camera_link</gz_frame_id>
-    </sensor>
-  </gazebo>
-</robot>
+/home/kimhoyun/DARAM-G/src/daramg_sim/urdf/RGB_D.xacro

File: install/daramg_sim/share/daramg_sim/urdf/imu.xacro (robot description, xacro)
@@ -1,20 +1 @@
-<?xml version="1.0"?>
-<robot xmlns:xacro="http://www.ros.org/wiki/xacro" name="robot_name">
-    <joint name="imu_joint" type="fixed">
-        <origin xyz="0 0 0" rpy="0 0 0" />
-        <parent link="base_link"/>
-        <child link="imu_link" />
-    </joint>
-    <link name="imu_link">
-    </link>
-    <gazebo reference="imu_link">
-        <sensor name="imu" type="imu">
-        <always_on>1</always_on>
-        <update_rate>50</update_rate>
-        <visualize>true</visualize>
-        <topic>imu</topic>
-        <enable_metrics>true</enable_metrics>
-        <gz_frame_id>imu_link</gz_frame_id>
-        </sensor>
-    </gazebo>
-</robot>
+/home/kimhoyun/DARAM-G/src/daramg_sim/urdf/imu.xacro

File: install/daramg_sim/share/daramg_sim/urdf/inertial_macros.xacro (robot description, xacro)
@@ -1,32 +1 @@
-<?xml version="1.0"?>
-<robot xmlns:xacro="http://www.ros.org/wiki/xacro" >
-    <!-- Specify some standard inertial calculations https://en.wikipedia.org/wiki/List_of_moments_of_inertia -->
-    <!-- These make use of xacro's mathematical functionality -->
-    <xacro:macro name="inertial_sphere" params="mass radius *origin">
-        <inertial>
-            <xacro:insert_block name="origin"/>
-            <mass value="${mass}" />
-            <inertia ixx="${(2/5) * mass * (radius*radius)}" ixy="0.0" ixz="0.0"
-                    iyy="${(2/5) * mass * (radius*radius)}" iyz="0.0"
-                    izz="${(2/5) * mass * (radius*radius)}" />
-        </inertial>
-    </xacro:macro>
-    <xacro:macro name="inertial_box" params="mass x y z *origin">
-        <inertial>
-            <xacro:insert_block name="origin"/>
-            <mass value="${mass}" />
-            <inertia ixx="${(1/12) * mass * (y*y+z*z)}" ixy="0.0" ixz="0.0"
-                    iyy="${(1/12) * mass * (x*x+z*z)}" iyz="0.0"
-                    izz="${(1/12) * mass * (x*x+y*y)}" />
-        </inertial>
-    </xacro:macro>
-    <xacro:macro name="inertial_cylinder" params="mass length radius *origin">
-        <inertial>
-            <xacro:insert_block name="origin"/>
-            <mass value="${mass}" />
-            <inertia ixx="${(1/12) * mass * (3*radius*radius + length*length)}" ixy="0.0" ixz="0.0"
-                    iyy="${(1/12) * mass * (3*radius*radius + length*length)}" iyz="0.0"
-                    izz="${(1/2) * mass * (radius*radius)}" />
-        </inertial>
-    </xacro:macro>
-</robot>
+/home/kimhoyun/DARAM-G/src/daramg_sim/urdf/inertial_macros.xacro

File: install/daramg_sim/share/daramg_sim/urdf/materials.xacro (robot description, xacro)
@@ -1,28 +1 @@
-<?xml version="1.0"?>
-<!-- This is the file for color implementation in RViz-->
-<robot>
-  <material name="black">
-    <color rgba="0.0 0.0 0.0 1.0"/>
-  </material>
-  <material name="white">
-    <color rgba="1.0 1.0 1.0 1.0"/>
-  </material>
-  <material name="red">
-    <color rgba="0.8 0.0 0.0 1.0"/>
-  </material>
-  <material name="blue">
-    <color rgba="0.0 0.0 0.8 1.0"/>
-  </material>
-  <material name="green">
-    <color rgba="0.0 0.8 0.0 1.0"/>
-  </material>
-  <material name="grey">
-    <color rgba="0.5 0.5 0.5 1.0"/>
-  </material>
-  <material name="orange">
-    <color rgba="${255/255} ${108/255} ${10/255} 1.0"/>
-  </material>
-  <material name="brown">
-    <color rgba="${222/255} ${207/255} ${195/255} 1.0"/>
-  </material>
-</robot>
+/home/kimhoyun/DARAM-G/src/daramg_sim/urdf/materials.xacro

File: src/daramg_sim/urdf/RGB_D.xacro (robot description, xacro)
@@ -60,8 +60,9 @@
     <sensor name="rgbd_camera" type="rgbd_camera">
       <camera>
-        <horizontal_fov>1.25</horizontal_fov>
+        <horizontal_fov>1.3962</horizontal_fov>
         <image>
-          <width>320</width>
-          <height>240</height>
+          <width>640</width>
+          <height>480</height>
+          <format>R8G8B8</format>
         </image>
         <clip>
@@ -75,5 +76,6 @@
       <visualize>true</visualize>
       <topic>camera</topic>
-      <gz_frame_id>camera_link</gz_frame_id>
+      <camera_info_topic>camera/camera_info</camera_info_topic>
+      <gz_frame_id>camera_link_optical</gz_frame_id>
     </sensor>
   </gazebo>
