Commit message: Migrate Simulation to Gazebo Classic

File: src/daramg_sim/urdf/2Dlidar.xacro (robot description, xacro)
@@ -25,40 +25,36 @@
         </visual>
     </link>
-  <gazebo reference="scan_link">
-    <sensor name="gpu_lidar" type="gpu_lidar">
-      <update_rate>10</update_rate>
-      <topic>scan</topic>
-      <gz_frame_id>scan_link</gz_frame_id>
-      <lidar>
-        <scan>
-          <horizontal>
-            <samples>720</samples>
-            <!--(max_angle-min_angle)/samples * resolution -->
-            <resolution>1</resolution>
-            <min_angle>-3.14156</min_angle>
-            <max_angle>3.14156</max_angle>
-          </horizontal>
-          <!-- Dirty hack for fake lidar detections with ogre 1 rendering in VM -->
-          <!-- <vertical>
-              <samples>3</samples>
-              <min_angle>-0.001</min_angle>
-              <max_angle>0.001</max_angle>
-          </vertical> -->
-        </scan>
-        <range>
-          <min>0.05</min>
-          <max>10.0</max>
-          <resolution>0.01</resolution>
-        </range>
-        <noise>
-            <type>gaussian</type>
+    <gazebo reference="scan_link">
+      <material>Gazebo/Grey</material>
+      <sensor type="ray" name="hokuyo_sensor">
+        <pose>0 0 0.0124 0 0 0</pose>
+        <visualize>false</visualize>
+        <update_rate>40</update_rate>
+        <ray>
+          <scan>
+            <horizontal>
+              <samples>1081</samples>
+              <resolution>1</resolution>
+              <min_angle>-2.3561944902</min_angle>
+              <max_angle>2.3561944902</max_angle>
+            </horizontal>
+          </scan>
+          <range>
+            <min>0.1</min>
+            <max>10.0</max>
+            <resolution>0.01</resolution>
+          </range>
+          <noise>
             <mean>0.0</mean>
             <stddev>0.01</stddev>
-        </noise>
-        <frame_id>scan_link</frame_id>
-      </lidar>
-      <always_on>1</always_on>
-      <visualize>true</visualize>
-    </sensor>
-  </gazebo>
+          </noise>
+        </ray>
+        <plugin name="gazebo_ros_hokuyo_controller" filename="libgazebo_ros_ray_sensor.so">
+          <ros>
+            <remapping>~/out:=scan</remapping>
+          </ros>
+          <output_type>sensor_msgs/LaserScan</output_type>
+        </plugin>
+      </sensor>
+    </gazebo>
 </robot>

File: src/daramg_sim/urdf/RGB_D.xacro (robot description, xacro)
@@ -57,26 +57,34 @@
     <link name="camera_link_optical">
     </link>
-  <gazebo reference="depth_link">
-    <sensor name="rgbd_camera" type="rgbd_camera">
-      <camera>
-        <horizontal_fov>1.3962</horizontal_fov>
-        <image>
-          <width>640</width>
-          <height>480</height>
-          <format>R8G8B8</format>
-        </image>
-        <clip>
-          <near>0.3</near>
-          <far>15</far>
-        </clip>
-        <optical_frame_id>camera_link_optical</optical_frame_id>
-      </camera>
-      <always_on>1</always_on>
-      <update_rate>20</update_rate>
-      <visualize>true</visualize>
-      <topic>camera</topic>
-      <camera_info_topic>camera/camera_info</camera_info_topic>
-      <gz_frame_id>camera_link_optical</gz_frame_id>
-    </sensor>
-  </gazebo>
+    <gazebo reference="depth_link">
+        <material>Gazebo/Blue</material>
+        <sensor name="camera" type="depth">
+            <pose> 0 0 0 0 0 0 </pose>
+            <visualize>true</visualize>
+            <update_rate>30</update_rate>
+            <camera>
+                <horizontal_fov>1.089</horizontal_fov>
+                <image>
+                    <format>B8G8R8</format>
+                    <width>640</width>
+                    <height>480</height>
+                </image>
+                <clip>
+                    <near>0.05</near>
+                    <far>8.0</far>
+                </clip>
+                <noise>
+                    <type>gaussian</type>
+                    <mean>0.0</mean>
+                    <stddev>0.007</stddev>
+                </noise>
+            </camera>
+            <plugin name="camera_controller" filename="libgazebo_ros_camera.so">
+                <frame_name>camera_link_optical</frame_name>
+                <min_depth>0.05</min_depth>
+                <max_depth>8.0</max_depth>
+                <updateRate>30.0</updateRate>
+            </plugin>
+        </sensor>
+    </gazebo>
 </robot>

File: src/daramg_sim/urdf/imu.xacro (robot description, xacro)
@@ -1,4 +1,4 @@
 <?xml version="1.0"?>
-<robot xmlns:xacro="http://www.ros.org/wiki/xacro" name="robot_name">
+<robot xmlns:xacro="http://www.ros.org/wiki/xacro">
     <joint name="imu_joint" type="fixed">
         <origin xyz="0 0 0" rpy="0 0 0" />
@@ -9,11 +9,59 @@
     </link>
     <gazebo reference="imu_link">
+        <gravity>true</gravity>
         <sensor name="imu" type="imu">
-        <always_on>1</always_on>
-        <update_rate>50</update_rate>
-        <visualize>true</visualize>
-        <topic>imu</topic>
-        <enable_metrics>true</enable_metrics>
-        <gz_frame_id>imu_link</gz_frame_id>
+            <always_on>true</always_on>
+            <update_rate>100</update_rate>
+            <visualize>true</visualize>
+            <topic>imu/data</topic>
+            <imu>
+                <angular_velocity>
+                    <x>
+                        <noise type="gaussian">
+                            <mean>0.0</mean>
+                            <stddev>2e-4</stddev>
+                        </noise>
+                    </x>
+                    <y>
+                        <noise type="gaussian">
+                            <mean>0.0</mean>
+                            <stddev>2e-4</stddev>
+                        </noise>
+                    </y>
+                    <z>
+                        <noise type="gaussian">
+                            <mean>0.0</mean>
+                            <stddev>2e-4</stddev>
+                        </noise>
+                    </z>
+                </angular_velocity>
+                <linear_acceleration>
+                    <x>
+                        <noise type="gaussian">
+                            <mean>0.0</mean>
+                            <stddev>1.7e-2</stddev>
+                        </noise>
+                    </x>
+                    <y>
+                        <noise type="gaussian">
+                            <mean>0.0</mean>
+                            <stddev>1.7e-2</stddev>
+                        </noise>
+                    </y>
+                    <z>
+                        <noise type="gaussian">
+                            <mean>0.0</mean>
+                            <stddev>1.7e-2</stddev>
+                        </noise>
+                    </z>
+                </linear_acceleration>
+            </imu>
+            <plugin name="imu" filename="libgazebo_ros_imu_sensor.so">
+                <ros>
+                    <namespace>imu</namespace>
+                    <remapping>~/out:=data</remapping>
+                </ros>
+                <initialOrientationAsReference>true</initialOrientationAsReference>
+            </plugin>
         </sensor>
     </gazebo>

Commit message: Add Gazebo Classic sim and Gazebo Harmonic Sim. In Gazebo Harmonic, We can do RTAB-MAP sim

File: src/daramg_sim/urdf/2Dlidar.xacro (robot description, xacro)
@@ -25,36 +25,40 @@
         </visual>
     </link>
-    <gazebo reference="scan_link">
-      <material>Gazebo/Grey</material>
-      <sensor type="ray" name="hokuyo_sensor">
-        <pose>0 0 0.0124 0 0 0</pose>
-        <visualize>false</visualize>
-        <update_rate>40</update_rate>
-        <ray>
-          <scan>
-            <horizontal>
-              <samples>1081</samples>
-              <resolution>1</resolution>
-              <min_angle>-2.3561944902</min_angle>
-              <max_angle>2.3561944902</max_angle>
-            </horizontal>
-          </scan>
-          <range>
-            <min>0.1</min>
-            <max>10.0</max>
-            <resolution>0.01</resolution>
-          </range>
-          <noise>
+  <gazebo reference="scan_link">
+    <sensor name="gpu_lidar" type="gpu_lidar">
+      <update_rate>10</update_rate>
+      <topic>scan</topic>
+      <gz_frame_id>scan_link</gz_frame_id>
+      <lidar>
+        <scan>
+          <horizontal>
+            <samples>720</samples>
+            <!--(max_angle-min_angle)/samples * resolution -->
+            <resolution>1</resolution>
+            <min_angle>-3.14156</min_angle>
+            <max_angle>3.14156</max_angle>
+          </horizontal>
+          <!-- Dirty hack for fake lidar detections with ogre 1 rendering in VM -->
+          <!-- <vertical>
+              <samples>3</samples>
+              <min_angle>-0.001</min_angle>
+              <max_angle>0.001</max_angle>
+          </vertical> -->
+        </scan>
+        <range>
+          <min>0.05</min>
+          <max>10.0</max>
+          <resolution>0.01</resolution>
+        </range>
+        <noise>
+            <type>gaussian</type>
             <mean>0.0</mean>
             <stddev>0.01</stddev>
-          </noise>
-        </ray>
-        <plugin name="gazebo_ros_hokuyo_controller" filename="libgazebo_ros_ray_sensor.so">
-          <ros>
-            <remapping>~/out:=scan</remapping>
-          </ros>
-          <output_type>sensor_msgs/LaserScan</output_type>
-        </plugin>
-      </sensor>
-    </gazebo>
+        </noise>
+        <frame_id>scan_link</frame_id>
+      </lidar>
+      <always_on>1</always_on>
+      <visualize>true</visualize>
+    </sensor>
+  </gazebo>
 </robot>

File: src/daramg_sim/urdf/imu.xacro (robot description, xacro)
@@ -1,4 +1,4 @@
 <?xml version="1.0"?>
-<robot xmlns:xacro="http://www.ros.org/wiki/xacro">
+<robot xmlns:xacro="http://www.ros.org/wiki/xacro" name="robot_name">
     <joint name="imu_joint" type="fixed">
         <origin xyz="0 0 0" rpy="0 0 0" />
@@ -9,59 +9,11 @@
     </link>
     <gazebo reference="imu_link">
-        <gravity>true</gravity>
         <sensor name="imu" type="imu">
-            <always_on>true</always_on>
-            <update_rate>100</update_rate>
-            <visualize>true</visualize>
-            <topic>imu/data</topic>
-            <imu>
-                <angular_velocity>
-                    <x>
-                        <noise type="gaussian">
-                            <mean>0.0</mean>
-                            <stddev>2e-4</stddev>
-                        </noise>
-                    </x>
-                    <y>
-                        <noise type="gaussian">
-                            <mean>0.0</mean>
-                            <stddev>2e-4</stddev>
-                        </noise>
-                    </y>
-                    <z>
-                        <noise type="gaussian">
-                            <mean>0.0</mean>
-                            <stddev>2e-4</stddev>
-                        </noise>
-                    </z>
-                </angular_velocity>
-                <linear_acceleration>
-                    <x>
-                        <noise type="gaussian">
-                            <mean>0.0</mean>
-                            <stddev>1.7e-2</stddev>
-                        </noise>
-                    </x>
-                    <y>
-                        <noise type="gaussian">
-                            <mean>0.0</mean>
-                            <stddev>1.7e-2</stddev>
-                        </noise>
-                    </y>
-                    <z>
-                        <noise type="gaussian">
-                            <mean>0.0</mean>
-                            <stddev>1.7e-2</stddev>
-                        </noise>
-                    </z>
-                </linear_acceleration>
-            </imu>
-            <plugin name="imu" filename="libgazebo_ros_imu_sensor.so">
-                <ros>
-                    <namespace>imu</namespace>
-                    <remapping>~/out:=data</remapping>
-                </ros>
-                <initialOrientationAsReference>true</initialOrientationAsReference>
-            </plugin>
+        <always_on>1</always_on>
+        <update_rate>50</update_rate>
+        <visualize>true</visualize>
+        <topic>imu</topic>
+        <enable_metrics>true</enable_metrics>
+        <gz_frame_id>imu_link</gz_frame_id>
         </sensor>
     </gazebo>

File: src/daramg_sim_classic/urdf/RGB_D.xacro (robot description, xacro)
@@ -3,5 +3,5 @@
     <!-- STEP 10 - Lidar -->
     <joint name="depth_pillar_joint" type="fixed">
-        <origin xyz="0.25 0.0 0.275" rpy="0.0 0.0 0.0"/>
+        <origin xyz="0.15 0.0 0.275" rpy="0.0 0.0 0.0"/>
         <parent link="base_link"/>
         <child link="depth_pillar"/>
@@ -57,24 +57,34 @@
     <link name="camera_link_optical">
     </link>
-  <gazebo reference="depth_link">
-    <sensor name="rgbd_camera" type="rgbd_camera">
-      <camera>
-        <horizontal_fov>1.25</horizontal_fov>
-        <image>
-          <width>320</width>
-          <height>240</height>
-        </image>
-        <clip>
-          <near>0.3</near>
-          <far>15</far>
-        </clip>
-        <optical_frame_id>camera_link_optical</optical_frame_id>
-      </camera>
-      <always_on>1</always_on>
-      <update_rate>20</update_rate>
-      <visualize>true</visualize>
-      <topic>camera</topic>
-      <gz_frame_id>camera_link_optical</gz_frame_id>
-    </sensor>
-  </gazebo>
+    <gazebo reference="depth_link">
+        <material>Gazebo/Blue</material>
+        <sensor name="camera" type="depth">
+            <pose> 0 0 0 0 0 0 </pose>
+            <visualize>true</visualize>
+            <update_rate>30</update_rate>
+            <camera>
+                <horizontal_fov>1.089</horizontal_fov>
+                <image>
+                    <format>B8G8R8</format>
+                    <width>640</width>
+                    <height>480</height>
+                </image>
+                <clip>
+                    <near>0.05</near>
+                    <far>8.0</far>
+                </clip>
+                <noise>
+                    <type>gaussian</type>
+                    <mean>0.0</mean>
+                    <stddev>0.007</stddev>
+                </noise>
+            </camera>
+            <plugin name="camera_controller" filename="libgazebo_ros_camera.so">
+                <frame_name>camera_link_optical</frame_name>
+                <min_depth>0.05</min_depth>
+                <max_depth>8.0</max_depth>
+                <updateRate>30.0</updateRate>
+            </plugin>
+        </sensor>
+    </gazebo>
 </robot>

Commit message: Add Path Planning and Control Package

File: src/daramg_sim/urdf/2Dlidar.xacro (robot description, xacro)
@@ -5,5 +5,5 @@
         <origin xyz="0.25 0 0.25" rpy="0 0 0"/>
         <child link="scan_link"/>
-        <parent link="base_link"/>
+        <parent link="base_footprint"/>
         <axis xyz="0 1 0" rpy="0 0 0"/>
     </joint>
@@ -48,5 +48,5 @@
         <range>
           <min>0.05</min>
-          <max>10.0</max>
+          <max>6.0</max>
           <resolution>0.01</resolution>
         </range>

File: src/daramg_sim/urdf/RGB_D.xacro (robot description, xacro)
@@ -4,5 +4,5 @@
     <joint name="depth_pillar_joint" type="fixed">
         <origin xyz="0.25 0.0 0.275" rpy="0.0 0.0 0.0"/>
-        <parent link="base_link"/>
+        <parent link="base_footprint"/>
         <child link="depth_pillar"/>
         <axis xyz="0.0 0.0 0.0"/>

File: src/daramg_sim/urdf/imu.xacro (robot description, xacro)
@@ -3,5 +3,5 @@
     <joint name="imu_joint" type="fixed">
         <origin xyz="0 0 0" rpy="0 0 0" />
-        <parent link="base_link"/>
+        <parent link="base_footprint"/>
         <child link="imu_link" />
     </joint>

File: src/daramg_sim/urdf/simple_rover.urdf (robot description, URDF)
Before this commit: robot simple_rover, 6 links, 5 joints
Links:
- removed link base_link
- added link base_footprint
Joints:
- joint chassis_joint: parent base_link -> base_footprint
- joint front_left_wheel_joint: parent base_link -> base_footprint
- joint front_right_wheel_joint: parent base_link -> base_footprint
- joint rear_left_wheel_joint: parent base_link -> base_footprint
- joint rear_right_wheel_joint: parent base_link -> base_footprint
