Commit message: Add simple robotic arm in rover

File: src/daramg_sim/urdf/simple_rover.urdf (robot description, URDF)
Before this commit: robot simple_rover, 6 links, 5 joints
Links:
- added link front_left_column; collision box size=0.06 0.06 0.30; visual box size=0.06 0.06 0.30
- added link front_right_column; collision box size=0.06 0.06 0.30; visual box size=0.06 0.06 0.30
- added link rear_left_column; collision box size=0.06 0.06 0.30; visual box size=0.06 0.06 0.30
- added link rear_right_column; collision box size=0.06 0.06 0.30; visual box size=0.06 0.06 0.30
Joints:
- added joint front_left_column_joint: type fixed, parent chassis, child front_left_column, origin xyz=0.25 0.20 0.30 rpy=0 0 0
- added joint front_right_column_joint: type fixed, parent chassis, child front_right_column, origin xyz=0.25 -0.20 0.30 rpy=0 0 0
- added joint rear_left_column_joint: type fixed, parent chassis, child rear_left_column, origin xyz=-0.25 0.20 0.30 rpy=0 0 0
- added joint rear_right_column_joint: type fixed, parent chassis, child rear_right_column, origin xyz=-0.25 -0.20 0.30 rpy=0 0 0
- joint chassis_joint: origin xyz=0.0 0.0 0.0 rpy=0.0 0.0 0.0 -> xyz=0 0 0 rpy=0 0 0
- joint front_left_wheel_joint: axis 0.0 1.0 0.0 -> 0 1 0; origin xyz=0.25 0.2 0.0 rpy=0.0 0.0 0.0 -> xyz=0 0 -0.20 rpy=0 0 0; parent base_footprint -> front_left_column
- joint front_right_wheel_joint: axis 0.0 1.0 0.0 -> 0 1 0; origin xyz=0.25 -0.2 0.0 rpy=0.0 0.0 0.0 -> xyz=0 0 -0.20 rpy=0 0 0; parent base_footprint -> front_right_column
- joint rear_left_wheel_joint: axis 0.0 1.0 0.0 -> 0 1 0; origin xyz=-0.25 0.2 0.0 rpy=0.0 0.0 0.0 -> xyz=0 0 -0.20 rpy=0 0 0; parent base_footprint -> rear_left_column
- joint rear_right_wheel_joint: axis 0.0 1.0 0.0 -> 0 1 0; origin xyz=-0.25 -0.2 0.0 rpy=0.0 0.0 0.0 -> xyz=0 0 -0.20 rpy=0 0 0; parent base_footprint -> rear_right_column
