Commit message: change simulation file

File: src/daramg_sim/urdf/ramgbot.urdf (robot description, URDF)
Before this commit: robot ramgbot, 6 links, 5 joints
Links:
- link chassis: geometry collision box size=0.3 0.3 0.15; visual box size=0.3 0.3 0.15
Joints:
- joint front_left_wheel_joint: origin xyz=0.15 0.15 -0.15 rpy=0 0 0 -> xyz=0.15 0.15 -0.12 rpy=0 0 0
- joint front_right_wheel_joint: origin xyz=0.15 -0.15 -0.15 rpy=0 0 0 -> xyz=0.15 -0.15 -0.12 rpy=0 0 0
- joint rear_left_wheel_joint: origin xyz=-0.15 0.15 -0.15 rpy=0 0 0 -> xyz=-0.15 0.15 -0.12 rpy=0 0 0
- joint rear_right_wheel_joint: origin xyz=-0.15 -0.15 -0.15 rpy=0 0 0 -> xyz=-0.15 -0.15 -0.12 rpy=0 0 0
